Commit message: add hj hand urdf
add hj_hand urdf

File: gripper_ur3/urdf/ar10.urdf.xacro (robot description, xacro)
@@ -12,5 +12,4 @@
 This model is outdated, for a more accurate representation, ar10.urdf is recommended instead. -->
 <robot xmlns:xacro="http://www.ros.org/wiki/xacro" name="ar10">
-  <xacro:macro name="ar10" params="prefix">
 <!--robot name="ar10"> -->
 <!--****************WRIST PLATE************************* -->
@@ -32,10 +31,4 @@
     </collision>
   </link>
-<!--****************MY editing************************* -->
-  <joint name="wrist2ee_link" type="fixed">
-    <parent link="${prefix}ee_link"/>
-    <child link="wrist_plate"/>
-    <origin xyz="0.008 0.0 0.0" rpy="${-pi/2} ${-pi} ${-pi/2}"/>
-  </joint>
 <!--****************CIRCUIT BOARD*************************-->
   <xacro:property name="circuit_support_x" value=".0555" />
@@ -269,91 +262,4 @@
     <mimic joint="pris2" multiplier="79.93" offset="0.29" />
   </joint>
-  <link name="finger2a">
-    <visual>
-      <geometry>
-        <box size="${fingera_x} ${fingera_y} ${fingera_z}"/>
-      </geometry>
-      <origin xyz="0 0 ${fingera_z/2}"/>
-      <material name="blue">
-      </material>
-    </visual>
-    <collision>
-      <geometry>
-        <box size="${fingera_x} ${fingera_y} ${fingera_z}"/>
-      </geometry>
-      <origin xyz="0 0 ${fingera_z/2}"/>
-    </collision>
-    <inertial>
-      <mass value="1"/>
-      <inertia ixx="0.4" ixy="0.0" ixz="0.0" iyy="0.4" iyz="0.0" izz="0.2"/>
-    </inertial>
-  </link>
-  <joint name="knuckle2_to_finger2a" type="revolute">
-    <axis xyz="-1 0 0"/>
-    <limit effort="1000.0" lower="0.0" upper="1.5" velocity="0.5"/>
-    <parent link="knuckle2"/>
-    <child link="finger2a"/>
-    <origin xyz="0 0 .02"/>
-    <joint_properties damping="1.0" friction="0.0"/>
-    <mimic joint="pris4" multiplier="79.93" offset="0.29" />
-  </joint>
-  <link name="finger3a">
-    <visual>
-      <geometry>
-        <box size="${fingera_x} ${fingera_y} ${fingera_z}"/>
-      </geometry>
-      <origin xyz="0 0 ${fingera_z/2}"/>
-      <material name="blue">
-      </material>
-    </visual>
-    <collision>
-      <geometry>
-        <box size="${fingera_x} ${fingera_y} ${fingera_z}"/>
-      </geometry>
-      <origin xyz="0 0 ${fingera_z/2}"/>
-    </collision>
-    <inertial>
-      <mass value="1"/>
-      <inertia ixx="0.4" ixy="0.0" ixz="0.0" iyy="0.4" iyz="0.0" izz="0.2"/>
-    </inertial>
-  </link>
-  <joint name="knuckle3_to_finger3a" type="revolute">
-    <axis xyz="-1 0 0"/>
-    <limit effort="1000.0" lower="0.0" upper="1.5" velocity="0.5"/>
-    <parent link="knuckle3"/>
-    <child link="finger3a"/>
-    <origin xyz="0 0 .03"/>
-    <joint_properties damping="1.0" friction="0.0"/>
-    <mimic joint="pris6" multiplier="79.93" offset="0.29" />
-  </joint>
-  <link name="finger4a">
-    <visual>
-      <geometry>
-        <box size="${fingera_x} ${fingera_y} ${fingera_z}"/>
-      </geometry>
-      <origin xyz="0 0 ${fingera_z/2}"/>
-      <material name="blue">
-      </material>
-    </visual>
-    <collision>
-      <geometry>
-        <box size="${fingera_x} ${fingera_y} ${fingera_z}"/>
-      </geometry>
-      <origin xyz="0 0 ${fingera_z/2}"/>
-    </collision>
-    <inertial>
-      <mass value="1"/>
-      <inertia ixx="0.4" ixy="0.0" ixz="0.0" iyy="0.4" iyz="0.0" izz="0.2"/>
-    </inertial>
-  </link>
-  <joint name="knuckle4_to_finger4a" type="revolute">
-    <axis xyz="-1 0 0"/>
-    <limit effort="1000.0" lower="0.0" upper="1.5" velocity="0.5"/>
-    <parent link="knuckle4"/>
-    <child link="finger4a"/>
-    <origin xyz="0 0 .03"/>
-    <joint_properties damping="1.0" friction="0.0"/>
-    <mimic joint="pris8" multiplier="79.93" offset="0.29" />
-  </joint>
   <link name="finger1b">
     <visual>
@@ -382,93 +288,6 @@
     <child link="finger1b"/>
     <origin xyz="0 0 ${fingera_z}"/>
-    <mimic joint="pris3" multiplier="79.64" offset="0.29" />
+    <mimic joint="pris2" multiplier="79.64" offset="0.29" />
     <joint_properties damping="1.0" friction="0.0"/>
-  </joint>
-  <link name="finger2b">
-    <visual>
-      <geometry>
-        <box size="${fingerb_x} ${fingerb_y} ${fingerb_z}"/>
-      </geometry>
-      <origin xyz="0 0 ${fingerb_z/2}"/>
-      <material name="blue">
-      </material>
-    </visual>
-    <collision>
-      <geometry>
-        <box size="${fingerb_x} ${fingerb_y} ${fingerb_z}"/>
-      </geometry>
-      <origin xyz="0 0 ${fingerb_z/2}"/>
-    </collision>
-    <inertial>
-      <mass value="1"/>
-      <inertia ixx="0.4" ixy="0.0" ixz="0.0" iyy="0.4" iyz="0.0" izz="0.2"/>
-    </inertial>
-  </link>
-  <joint name="finger2a_to_finger2b" type="revolute">
-    <axis xyz="-1 0 0"/>
-    <limit effort="1000.0" lower="0.0" upper="1.5" velocity="0.5"/>
-    <parent link="finger2a"/>
-    <child link="finger2b"/>
-    <origin xyz="0 0 ${fingera_z}"/>
-    <joint_properties damping="1.0" friction="0.0"/>
-    <mimic joint="pris5" multiplier="79.64" offset="0.29" />
-  </joint>
-  <link name="finger3b">
-    <visual>
-      <geometry>
-        <box size="${fingerb_x} ${fingerb_y} ${fingerb_z}"/>
-      </geometry>
-      <origin xyz="0 0 ${fingerb_z/2}"/>
-      <material name="blue">
-      </material>
-    </visual>
-    <collision>
-      <geometry>
-        <box size="${fingerb_x} ${fingerb_y} ${fingerb_z}"/>
-      </geometry>
-      <origin xyz="0 0 ${fingerb_z/2}"/>
-    </collision>
-    <inertial>
-      <mass value="1"/>
-      <inertia ixx="0.4" ixy="0.0" ixz="0.0" iyy="0.4" iyz="0.0" izz="0.2"/>
-    </inertial>
-  </link>
-  <joint name="finger3a_to_finger3b" type="revolute">
-    <axis xyz="-1 0 0"/>
-    <limit effort="1000.0" lower="0.0" upper="1.5" velocity="0.5"/>
-    <parent link="finger3a"/>
-    <child link="finger3b"/>
-    <origin xyz="0 0 ${fingera_z}"/>
-    <joint_properties damping="1.0" friction="0.0"/>
-    <mimic joint="pris7" multiplier="79.64" offset="0.29" />
-  </joint>
-  <link name="finger4b">
-    <visual>
-      <geometry>
-        <box size="${fingerb_x} ${fingerb_y} ${fingerb_z}"/>
-      </geometry>
-      <origin xyz="0 0 ${fingerb_z/2}"/>
-      <material name="blue">
-      </material>
-    </visual>
-    <collision>
-      <geometry>
-        <box size="${fingerb_x} ${fingerb_y} ${fingerb_z}"/>
-      </geometry>
-      <origin xyz="0 0 ${fingerb_z/2}"/>
-    </collision>
-    <inertial>
-      <mass value="1"/>
-      <inertia ixx="0.4" ixy="0.0" ixz="0.0" iyy="0.4" iyz="0.0" izz="0.2"/>
-    </inertial>
-  </link>
-  <joint name="finger4a_to_finger4b" type="revolute">
-    <axis xyz="-1 0 0"/>
-    <limit effort="1000.0" lower="0.0" upper="1.5" velocity="0.5"/>
-    <parent link="finger4a"/>
-    <child link="finger4b"/>
-    <origin xyz="0 0 ${fingera_z}"/>
-    <joint_properties damping="1.0" friction="0.0"/>
-    <mimic joint="pris9" multiplier="79.64" offset="0.29" />
   </joint>
   <link name="finger1c">
@@ -498,92 +317,5 @@
     <axis xyz="-1 0 0"/>
     <limit effort="1000.0" lower="0" upper="1.5" velocity="0.5"/>
-    <mimic joint="pris3" multiplier="68.88" offset="0.16" />
-  </joint>
-  <link name="finger2c">
-    <visual>
-      <geometry>
-        <box size="${fingerc_x} ${fingerc_y} ${fingerc_z}"/>
-      </geometry>
-      <origin xyz="0 0 ${fingerc_z/2}"/>
-      <material name="black">
-      </material>
-    </visual>
-    <collision>
-      <geometry>
-        <box size="${fingerc_x} ${fingerc_y} ${fingerc_z}"/>
-      </geometry>
-      <origin xyz="0 0 ${fingerb_z}"/>
-    </collision>
-    <inertial>
-      <mass value="1"/>
-      <inertia ixx="0.4" ixy="0.0" ixz="0.0" iyy="0.4" iyz="0.0" izz="0.2"/>
-    </inertial>
-  </link>
-  <joint name="finger2b_to_finger2c" type="revolute">
-    <parent link="finger2b"/>
-    <child link="finger2c"/>
-    <origin xyz="0 0 ${fingerb_z}"/>
-    <axis xyz="-1 0 0"/>
-    <limit effort="1000.0" lower="0" upper="1.5" velocity="0.5"/>
-    <mimic joint="pris5" multiplier="68.88" offset="0.16" />
-  </joint>
-  <link name="finger3c">
-    <visual>
-      <geometry>
-        <box size="${fingerc_x} ${fingerc_y} ${fingerc_z}"/>
-      </geometry>
-      <origin xyz="0 0 ${fingerc_z/2}"/>
-      <material name="black">
-      </material>    <inertial>
-      <mass value="10"/>
-      <inertia ixx="0.4" ixy="0.0" ixz="0.0" iyy="0.4" iyz="0.0" izz="0.2"/>
-    </inertial>
-    </visual>
-    <collision>
-      <geometry>
-        <box size="${fingerc_x} ${fingerc_y} ${fingerc_z}"/>
-      </geometry>
-      <origin xyz="0 0 ${fingerc_z/2}"/>
-    </collision>
-    <inertial>
-      <mass value="1"/>
-      <inertia ixx="0.4" ixy="0.0" ixz="0.0" iyy="0.4" iyz="0.0" izz="0.2"/>
-    </inertial>
-  </link>
-  <joint name="finger3b_to_finger3c" type="revolute">
-    <parent link="finger3b"/>
-    <child link="finger3c"/>
-    <origin xyz="0 0 ${fingerb_z}"/>
-    <axis xyz="-1 0 0"/>
-    <limit effort="1000.0" lower="0" upper="1.5" velocity="0.5"/>
-    <mimic joint="pris7" multiplier="68.88" offset="0.16" />
-  </joint>
-  <link name="finger4c">
-    <visual>
-      <geometry>
-        <box size="${fingerc_x} ${fingerc_y} ${fingerc_z}"/>
-      </geometry>
-      <origin xyz="0 0 ${fingerc_z/2}"/>
-      <material name="black">
-      </material>
-    </visual>
-    <collision>
-      <geometry>
-        <box size="${fingerc_x} ${fingerc_y} ${fingerc_z}"/>
-      </geometry>
-      <origin xyz="0 0 ${fingerc_z/2}"/>
-    </collision>
-    <inertial>
-      <mass value="1"/>
-      <inertia ixx="0.4" ixy="0.0" ixz="0.0" iyy="0.4" iyz="0.0" izz="0.2"/>
-    </inertial>
-  </link>
-  <joint name="finger4b_to_finger4c" type="revolute">
-    <parent link="finger4b"/>
-    <child link="finger4c"/>
-    <origin xyz="0 0 ${fingerb_z}"/>
-    <axis xyz="-1 0 0"/>
-    <limit effort="1000.0" lower="0" upper="1.5" velocity="0.5"/>
-    <mimic joint="pris9" multiplier="68.88" offset="0.19" />
+    <mimic joint="pris2" multiplier="68.88" offset="0.16" />
   </joint>
 <!--****************THUMB*************************-->
@@ -829,333 +561,3 @@
     <origin xyz="0 .03 0" rpy = "1.57 0 0"/>
   </joint>
-  <link name="motor3">
-    <visual>
-      <geometry>
-        <box size="${motor_x} ${motor_y} ${motor_z}"/>
-      </geometry>
-      <origin xyz="0 .02 0"/>
-      <material name="black">
-      </material>
-    </visual>
-    <collision>
-      <geometry>
-        <box size="${motor_x} ${motor_y} ${motor_z}"/>
-      </geometry>
-      <origin xyz="0 .02 0"/>
-    </collision>
-    <inertial>
-      <mass value="1"/>
-      <inertia ixx="0.4" ixy="0.0" ixz="0.0" iyy="0.4" iyz="0.0" izz="0.2"/>
-    </inertial>
-  </link>
-  <joint name="motor3_to_finger1a" type="fixed">
-    <axis xyz="1 0 0"/>
-    <parent link="finger1a"/>
-    <child link="motor3"/>
-    <origin xyz="0 -.0145 .01" rpy = "1.57 0 0"/>
-  </joint>
-  <link name="pris3">
-    <visual>
-      <geometry>
-        <box size="${pris_x} ${pris_y} ${pris_z}"/>
-      </geometry>
-      <origin xyz="0 0 0"/>
-      <material name="black">
-      </material>
-    </visual>
-    <inertial>
-      <mass value="1"/>
-      <inertia ixx="0.4" ixy="0.0" ixz="0.0" iyy="0.4" iyz="0.0" izz="0.2"/>
-    </inertial>
-  </link>
-  <joint name="pris3" type="prismatic">
-    <axis xyz="0 0 -1"/>
-    <limit effort="1000.0" lower="0.0" upper="0.02" velocity="0.1"/>
-    <parent link="motor3"/>
-    <child link="pris3"/>
-    <origin xyz="0 .03 0" rpy = "1.57 0 0"/>
-  </joint>
-  <link name="motor4">
-    <visual>
-      <geometry>
-        <box size="${motor_x} ${motor_y} ${motor_z}"/>
-      </geometry>
-      <origin xyz="0 .02 0"/>
-      <material name="black">
-      </material>
-    </visual>
-    <collision>
-      <geometry>
-        <box size="${motor_x} ${motor_y} ${motor_z}"/>
-      </geometry>
-      <origin xyz="0 .02 0"/>
-    </collision>
-    <inertial>
-      <mass value="1"/>
-      <inertia ixx="0.4" ixy="0.0" ixz="0.0" iyy="0.4" iyz="0.0" izz="0.2"/>
-    </inertial>
-  </link>
-  <joint name="knuckle2_to_motor4" type="fixed">
-    <axis xyz="1 0 0"/>
-    <parent link="knuckle2"/>
-    <child link="motor4"/>
-    <origin xyz="0 -.0145 -.045" rpy = "1.57 0 0"/>
-  </joint>
-  <link name="pris4">
-    <visual>
-      <geometry>
-        <box size="${pris_x} ${pris_y} ${pris_z}"/>
-      </geometry>
-      <origin xyz="0 0 0"/>
-      <material name="black">
-      </material>
-    </visual>
-    <inertial>
-      <mass value="1"/>
-      <inertia ixx="0.4" ixy="0.0" ixz="0.0" iyy="0.4" iyz="0.0" izz="0.2"/>
-    </inertial>
-  </link>
-  <joint name="pris4" type="prismatic">
-    <axis xyz="0 0 -1"/>
-    <limit effort="1000.0" lower="0.0" upper="0.02" velocity="0.1"/>
-    <parent link="motor4"/>
-    <child link="pris4"/>
-    <origin xyz="0 .03 0" rpy = "1.57 0 0"/>
-  </joint>
-  <link name="motor5">
-    <visual>
-      <geometry>
-        <box size="${motor_x} ${motor_y} ${motor_z}"/>
-      </geometry>
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