Commit message: update hand
2019.08.01 update

File: gripper_ur3/urdf/hj_hand.urdf.xacro (robot description, xacro)
@@ -1,5 +1,11 @@
 <?xml version="1.0"?>
 <robot xmlns:xacro="http://www.ros.org/wiki/xacro" name="hj_hand">
-<!--robot name="ar10"> -->
+<xacro:macro name="hj_hand" params="parent *origin">
+      <!--
+      Autor: Hyeonjun Park
+      2019.07.17
+      -->
+      <xacro:include filename="$(find gripper_ur3)/urdf/hj_hand_transmission.xacro" />
+      <xacro:include filename="$(find gripper_ur3)/urdf/hj_hand_gazebo.xacro" />
       <xacro:property name="motor_x" value="0.016" />
       <xacro:property name="motor_y" value="0.035" />
@@ -8,14 +14,14 @@
       <xacro:property name="pris_y" value="0.005" />
       <xacro:property name="pris_z" value="0.025" />
+      <xacro:property name="knucle_mass" value="0.010" />
+      <xacro:property name="MCP_mass" value="0.0125" />
+      <xacro:property name="PIP_mass" value="0.0125" />
+      <xacro:property name="DIP_mass" value="0.0025" />
+      <xacro:property name="motor_mass" value="0.015" />
       <xacro:property name="motor_joint_x" value="0.0" />
       <xacro:property name="motor_joint_y" value="-0.0145" />
       <xacro:property name="motor_joint_z" value="0.006" />
       <xacro:property name="eef_offset_z" value="0.025725" />
-      <link name="hj_hand_world" />
-      <joint name="hj_hand_world_joint" type="fixed">
-            <parent link="hj_hand_world"/>
-            <child link="wrist_plate"/>
-            <origin xyz="0.0 0.0 0.0" rpy="0.0 0.0 0.0"/>
-      </joint>
+      <xacro:property name="motor_max_upper" value="0.0103" /> <!--joint origin-->
 <!--****************WRIST PLATE************************* -->
       <link name="wrist_plate">
@@ -36,4 +42,10 @@
             </collision>
       </link>
+      <joint name="wrist_plate_joint" type="fixed">
+            <xacro:insert_block name="origin" />
+            <parent link="${parent}"/>
+            <child link="wrist_plate"/>
+            <limit lower="0.0" upper="0.0" effort="0.0" velocity="0.0"/>
+      </joint>
       <!--**************** hand palm*************************-->
       <xacro:property name="hand_palm_x" value="0.0" />
@@ -60,9 +72,11 @@
             </collision>
             <inertial>
-                  <mass value="1"/>
-                  <inertia ixx="0.4" ixy="0.0" ixz="0.0" iyy="0.4" iyz="0.0" izz="0.2"/>
-            </inertial>
-      </link>
-      <joint name="wrist_plate_to_hand_palm" type="fixed">
+                  <mass value="0.09"/>
+                  <inertia ixx="1.0e-03" ixy="0.0" ixz="0.0"
+               iyy="1.0e-03" iyz="0.0"
+               izz="1.0e-03" />
+            </inertial>
+      </link>
+      <joint name="hand_wrist_plate_to_hand_palm" type="fixed">
             <parent link="wrist_plate"/>
             <child link="hand_palm"/>
@@ -92,9 +106,11 @@
       </collision>
       <inertial>
-            <mass value="1"/>
-            <inertia ixx="0.4" ixy="0.0" ixz="0.0" iyy="0.4" iyz="0.0" izz="0.2"/>
-      </inertial>
-      </link>
-      <joint name="hand_palm_to_knuckle_index" type="fixed">
+            <mass value="${knucle_mass}"/>
+            <inertia ixx="1.0e-03" ixy="0.0" ixz="0.0"
+               iyy="1.0e-03" iyz="0.0"
+               izz="1.0e-03" />
+      </inertial>
+      </link>
+      <joint name="knuckle_index_joint" type="fixed">
       <parent link="hand_palm"/>
       <child link="knuckle_index"/>
@@ -119,9 +135,11 @@
       </collision>
       <inertial>
-            <mass value="1"/>
-            <inertia ixx="0.4" ixy="0.0" ixz="0.0" iyy="0.4" iyz="0.0" izz="0.2"/>
-      </inertial>
-      </link>
-            <joint name="hand_palm_to_knuckle_middle" type="fixed">
+            <mass value="${knucle_mass}"/>
+            <inertia ixx="1.0e-03" ixy="0.0" ixz="0.0"
+               iyy="1.0e-03" iyz="0.0"
+               izz="1.0e-03" />
+      </inertial>
+      </link>
+            <joint name="knuckle_middle_joint" type="fixed">
             <parent link="hand_palm"/>
             <child link="knuckle_middle"/>
@@ -146,9 +164,11 @@
             </collision>
             <inertial>
-                  <mass value="1"/>
-                  <inertia ixx="0.4" ixy="0.0" ixz="0.0" iyy="0.4" iyz="0.0" izz="0.2"/>
-            </inertial>
-      </link>
-            <joint name="hand_palm_to_knuckle_ring" type="fixed">
+                  <mass value="${knucle_mass}"/>
+                  <inertia ixx="1.0e-03" ixy="0.0" ixz="0.0"
+               iyy="1.0e-03" iyz="0.0"
+               izz="1.0e-03" />
+            </inertial>
+      </link>
+            <joint name="knuckle_ring_joint" type="fixed">
                   <parent link="hand_palm"/>
                   <child link="knuckle_ring"/>
@@ -173,9 +193,11 @@
             </collision>
             <inertial>
-                  <mass value="1"/>
-                  <inertia ixx="0.4" ixy="0.0" ixz="0.0" iyy="0.4" iyz="0.0" izz="0.2"/>
-            </inertial>
-      </link>
-      <joint name="hand_palm_to_knuckle_little" type="fixed">
+                  <mass value="${knucle_mass}"/>
+                  <inertia ixx="1.0e-03" ixy="0.0" ixz="0.0"
+               iyy="1.0e-03" iyz="0.0"
+               izz="1.0e-03" />
+            </inertial>
+      </link>
+      <joint name="knuckle_little_joint" type="fixed">
             <parent link="hand_palm"/>
             <child link="knuckle_little"/>
@@ -228,9 +250,11 @@
             </collision>
             <inertial>
-                  <mass value="1"/>
-                  <inertia ixx="0.4" ixy="0.0" ixz="0.0" iyy="0.4" iyz="0.0" izz="0.2"/>
-            </inertial>
-      </link>
-      <joint name="hand_palm_to_knuckle_thumb" type="fixed">
+                  <mass value="${knucle_mass}"/>
+                  <inertia ixx="1.0e-03" ixy="0.0" ixz="0.0"
+               iyy="1.0e-03" iyz="0.0"
+               izz="1.0e-03" />
+            </inertial>
+      </link>
+      <joint name="knuckle_thumb_joint" type="fixed">
             <parent link="hand_palm"/>
             <child link="knuckle_thumb"/>
@@ -256,9 +280,11 @@
       </collision>
       <inertial>
-            <mass value="1"/>
-            <inertia ixx="0.4" ixy="0.0" ixz="0.0" iyy="0.4" iyz="0.0" izz="0.2"/>
-      </inertial>
-      </link>
-      <joint name="knuckle_thumb_joint_to_thumb_joint" type="revolute">
+            <mass value="${motor_mass}"/>
+            <inertia ixx="1.0e-03" ixy="0.0" ixz="0.0"
+               iyy="1.0e-03" iyz="0.0"
+               izz="1.0e-03" />
+      </inertial>
+      </link>
+      <joint name="thumb_jo_joint" type="revolute">
             <axis xyz="0 0 -1"/>    <!--z axis rotate -->
             <limit effort="1000.0" lower="0.0" upper="1.8" velocity="0.5"/>
@@ -288,9 +314,11 @@
       </collision>
       <inertial>
-            <mass value="1"/>
-            <inertia ixx="0.4" ixy="0.0" ixz="0.0" iyy="0.4" iyz="0.0" izz="0.2"/>
-      </inertial>
-      </link>
-      <joint name="thumb_joint_to_thumb_MCP" type="revolute">
+            <mass value="${MCP_mass}"/>
+            <inertia ixx="1.0e-03" ixy="0.0" ixz="0.0"
+               iyy="1.0e-03" iyz="0.0"
+               izz="1.0e-03" />
+      </inertial>
+      </link>
+      <joint name="thumb_MCP_joint" type="revolute">
             <axis xyz="0 1 0"/>
             <limit effort="1000.0" lower="0.0" upper="1.0" velocity="0.5"/>
@@ -320,9 +348,11 @@
       </collision>
       <inertial>
-            <mass value="1"/>
-            <inertia ixx="0.4" ixy="0.0" ixz="0.0" iyy="0.4" iyz="0.0" izz="0.2"/>
-      </inertial>
-      </link>
-      <joint name="thumb_MCP_to_thumb_DIP" type="revolute">
+            <mass value="${DIP_mass}"/>
+            <inertia ixx="1.0e-03" ixy="0.0" ixz="0.0"
+               iyy="1.0e-03" iyz="0.0"
+               izz="1.0e-03" />
+      </inertial>
+      </link>
+      <joint name="thumb_DIP_joint" type="revolute">
             <axis xyz="0 1 0"/>
             <limit effort="1000.0" lower="0.0" upper="0.8" velocity="0.5"/>
@@ -366,16 +396,18 @@
                   </material>
             </visual>
-            <collision>
+            <!--collision>
                   <geometry>
                   <box size="${motor_x} ${motor_y} ${motor_z}"/>
                   </geometry>
                   <origin xyz="0 .02 0"/>
-            </collision>
-            <inertial>
-                  <mass value="1"/>
-                  <inertia ixx="0.4" ixy="0.0" ixz="0.0" iyy="0.4" iyz="0.0" izz="0.2"/>
-            </inertial>
-      </link>
-      <joint name="knuckle_thumb_to_motor_thumb_jo" type="fixed">
+            </collision-->
+            <inertial>
+                  <mass value="${motor_mass}"/>
+                  <inertia ixx="1.0e-03" ixy="0.0" ixz="0.0"
+               iyy="1.0e-03" iyz="0.0"
+               izz="1.0e-03" />
+            </inertial>
+      </link>
+      <joint name="motor_thumb_jo_joint" type="fixed">
             <axis xyz="1 0 0"/>
             <parent link="knuckle_thumb"/>
@@ -393,11 +425,13 @@
             </visual>
             <inertial>
-                  <mass value="1"/>
-                  <inertia ixx="0.4" ixy="0.0" ixz="0.0" iyy="0.4" iyz="0.0" izz="0.2"/>
+                  <mass value="0.001"/>
+                  <inertia ixx="1.0e-03" ixy="0.0" ixz="0.0"
+               iyy="1.0e-03" iyz="0.0"
+               izz="1.0e-03" />
             </inertial>
       </link>
       <joint name="pris_thumb_jo_joint" type="prismatic">
             <axis xyz="0 0 -1"/>
-            <limit effort="1000.0" lower="0.0" upper="0.01" velocity="0.1"/>
+            <limit effort="1000.0" lower="0.0" upper="${motor_max_upper}" velocity="0.1"/>
             <parent link="motor_thumb_jo"/>
             <child link="pris_thumb_jo"/>
@@ -415,16 +449,18 @@
                   </material>
             </visual>
-            <collision>
+            <!--collision>
                   <geometry>
                   <box size="${motor_x} ${motor_y} ${motor_z}"/>
                   </geometry>
                   <origin xyz="0 .02 0"/>
-            </collision>
-            <inertial>
-                  <mass value="1"/>
-                  <inertia ixx="0.4" ixy="0.0" ixz="0.0" iyy="0.4" iyz="0.0" izz="0.2"/>
-            </inertial>
-      </link>
-      <joint name="thumb_joint_to_motor_thumb_DIP" type="fixed">
+            </collision-->
+            <inertial>
+                  <mass value="${DIP_mass}"/>
+                  <inertia ixx="1.0e-03" ixy="0.0" ixz="0.0"
+               iyy="1.0e-03" iyz="0.0"
+               izz="1.0e-03" />
+            </inertial>
+      </link>
+      <joint name="motor_thumb_DIP_joint" type="fixed">
             <axis xyz="1 0 0"/>
             <parent link="thumb_joint"/>
@@ -443,11 +479,13 @@
             </visual>
             <inertial>
-                  <mass value="1"/>
-                  <inertia ixx="0.4" ixy="0.0" ixz="0.0" iyy="0.4" iyz="0.0" izz="0.2"/>
+                  <mass value="0.001"/>
+                  <inertia ixx="1.0e-03" ixy="0.0" ixz="0.0"
+               iyy="1.0e-03" iyz="0.0"
+               izz="1.0e-03" />
             </inertial>
       </link>
       <joint name="pris_thumb_DIP_joint" type="prismatic">
             <axis xyz="0 0 -1"/>
-            <limit effort="1000.0" lower="0.0" upper="0.01" velocity="0.1"/>
+            <limit effort="1000.0" lower="0.0" upper="${motor_max_upper}" velocity="0.1"/>
             <parent link="motor_thumb_DIP"/>
             <child link="pris_thumb_DIP"/>
@@ -495,9 +533,11 @@
       </collision>
       <inertial>
-            <mass value="1"/>
-            <inertia ixx="0.4" ixy="0.0" ixz="0.0" iyy="0.4" iyz="0.0" izz="0.2"/>
-      </inertial>
-      </link>
-      <joint name="knuckle_index_to_index_MCP" type="revolute">
+            <mass value="${MCP_mass}"/>
+            <inertia ixx="1.0e-03" ixy="0.0" ixz="0.0"
+               iyy="1.0e-03" iyz="0.0"
+               izz="1.0e-03" />
+      </inertial>
+      </link>
+      <joint name="index_MCP_joint" type="revolute">
             <axis xyz="-1 0 0"/>
             <limit effort="1000.0" lower="0.0" upper="1.3" velocity="0.5"/>
@@ -529,9 +569,11 @@
       </collision>
       <inertial>
-            <mass value="1"/>
-            <inertia ixx="0.4" ixy="0.0" ixz="0.0" iyy="0.4" iyz="0.0" izz="0.2"/>
-      </inertial>
-      </link>
-      <joint name="index_MCP_to_index_PIP" type="revolute">
+            <mass value="${PIP_mass}"/>
+            <inertia ixx="1.0e-03" ixy="0.0" ixz="0.0"
+               iyy="1.0e-03" iyz="0.0"
+               izz="1.0e-03" />
+      </inertial>
+      </link>
+      <joint name="index_PIP_joint" type="revolute">
             <axis xyz="-1 0 0"/>
             <limit effort="1000.0" lower="0.0" upper="1.0" velocity="0.5"/>
@@ -564,9 +606,11 @@
       </collision>
       <inertial>
-            <mass value="1"/>
-            <inertia ixx="0.4" ixy="0.0" ixz="0.0" iyy="0.4" iyz="0.0" izz="0.2"/>
-      </inertial>
-      </link>
-      <joint name="index_PIP_to_index_DIP" type="revolute">
+            <mass value="${DIP_mass}"/>
+            <inertia ixx="1.0e-03" ixy="0.0" ixz="0.0"
+               iyy="1.0e-03" iyz="0.0"
+               izz="1.0e-03" />
+      </inertial>
+      </link>
+      <joint name="index_DIP_joint" type="revolute">
             <axis xyz="-1 0 0"/>
             <limit effort="1000.0" lower="0.0" upper="1.0" velocity="0.5"/>
@@ -610,9 +654,11 @@
       </collision>
       <inertial>
-            <mass value="1"/>
-            <inertia ixx="0.4" ixy="0.0" ixz="0.0" iyy="0.4" iyz="0.0" izz="0.2"/>
-      </inertial>
-      </link>
-      <joint name="knuckle_middle_to_middle_MCP" type="revolute">
+            <mass value="${MCP_mass}"/>
+            <inertia ixx="1.0e-03" ixy="0.0" ixz="0.0"
+               iyy="1.0e-03" iyz="0.0"
+               izz="1.0e-03" />
+      </inertial>
+      </link>
+      <joint name="middle_MCP_joint" type="revolute">
             <axis xyz="-1 0 0"/>
             <limit effort="1000.0" lower="0.0" upper="1.3" velocity="0.5"/>
@@ -644,9 +690,11 @@
       </collision>
       <inertial>
-            <mass value="1"/>
-            <inertia ixx="0.4" ixy="0.0" ixz="0.0" iyy="0.4" iyz="0.0" izz="0.2"/>
-      </inertial>
-      </link>
-      <joint name="middle_MCP_to_middle_PIP" type="revolute">
+            <mass value="${PIP_mass}"/>
+            <inertia ixx="1.0e-03" ixy="0.0" ixz="0.0"
+               iyy="1.0e-03" iyz="0.0"
+               izz="1.0e-03" />
+      </inertial>
+      </link>
+      <joint name="middle_PIP_joint" type="revolute">
             <axis xyz="-1 0 0"/>
             <limit effort="1000.0" lower="0.0" upper="1.0" velocity="0.5"/>
@@ -678,9 +726,11 @@
       </collision>
       <inertial>
-            <mass value="1"/>
-            <inertia ixx="0.4" ixy="0.0" ixz="0.0" iyy="0.4" iyz="0.0" izz="0.2"/>
-      </inertial>
-      </link>
-      <joint name="middle_PIP_to_middle_DIP" type="revolute">
+            <mass value="${DIP_mass}"/>
+            <inertia ixx="1.0e-03" ixy="0.0" ixz="0.0"
+               iyy="1.0e-03" iyz="0.0"
+               izz="1.0e-03" />
+      </inertial>
+      </link>
+      <joint name="middle_DIP_joint" type="revolute">
             <axis xyz="-1 0 0"/>
             <limit effort="1000.0" lower="0.0" upper="1.0" velocity="0.5"/>
@@ -724,9 +774,11 @@
       </collision>
       <inertial>
-            <mass value="1"/>
-            <inertia ixx="0.4" ixy="0.0" ixz="0.0" iyy="0.4" iyz="0.0" izz="0.2"/>
-      </inertial>
-      </link>
-      <joint name="knuckle_ring_to_ring_MCP" type="revolute">
+            <mass value="${MCP_mass}"/>
+            <inertia ixx="1.0e-03" ixy="0.0" ixz="0.0"
+               iyy="1.0e-03" iyz="0.0"
+               izz="1.0e-03" />
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